File: Main/Main.kicad_sch (KiCad schematic)
At the start: 0 parts

Commit message: Add files via upload
Other:
- note added: "104 - APA102 LED's"
- note added: "104 KEY FULL SIZE LAYOUT KEYS DIRECTLY TIED TO 74HC561 PARALLEL-IN, SERIAL-OUT (PISO) SHIFT REGISTER FOR SCANNING"
- note added: "5VDC, 2A TPS54231 BUCK CONVERTER POWERS: APA102 LED's, USB2514 HUB 3.3VDC, 1A TPS62130 BUCK CONVERTER POWERS: RM4A1 uC, STM32G431 uC, KEYS, E-INK"
- note added: "RENESAS RM4A1"
- note added: "USB-C PD PORT (9VDC, 3A)"
- note removed: "1.2VDC 500mA"
- note removed: "12VDC 500mA"
- note removed: "3.3VDC 500mA"
- note removed: "5VDC 1000mA"
Changed lines of the file:
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@@
+		)
+	)
+	(text "RENESAS RM4A1"
+		(exclude_from_sim no)
+		(at 292.1 127 0)
+		(effects
+			(font
+				(size 2.54 2.54)
+			)
 		)
 	)
@@
 		)
 	)
-	(text "5VDC\n1000mA"
-		(exclude_from_sim no)
-		(at 197.104 75.946 0)
+	(text "Serial"
+		(exclude_from_sim no)
+		(at 292.862 146.558 0)
+		(effects
+			(font
+				(size 1.27 1.27)
+			)
+			(justify left)
+		)
+	)
+	(text "USB 3.1 4 PORT CONTROLLER\nINPUT: TYPE C\nOUTPUT: 2 x TYPE C, 2 x USB A 2.0\nIC: USB7002T-I/KDX"
+		(exclude_from_sim no)
+		(at 217.17 38.354 0)
+		(effects
+			(font
+				(size 2.54 2.54)
+			)
+		)
+	)
+	(text "104 - APA102 LED's"
+		(exclude_from_sim no)
+		(at 292.1 203.2 0)
+		(effects
+			(font
+				(size 2.54 2.54)
+			)
+		)
+	)
+	(text "USB-C PD\nPORT\n(9VDC, 3A)"
+		(exclude_from_sim no)
+		(at 38.1 44.958 0)
 		(effects
 			(font
 				(face "Comic Sans MS")
-				(size 1.27 1.27)
-			)
-		)
-	)
-	(text "Serial"
-		(exclude_from_sim no)
-		(at 292.862 146.558 0)
-		(effects
-			(font
-				(size 1.27 1.27)
-			)
-			(justify left)
-		)
-	)
-	(text "USB 3.1 4 PORT CONTROLLER\nINPUT: TYPE C\nOUTPUT: 2 x TYPE C, 2 x USB A 2.0\nIC: USB7002T-I/KDX"
-		(exclude_from_sim no)
-		(at 217.17 38.354 0)
+				(size 1.905 1.905)
+			)
+		)
+	)
+	(text "104 KEY FULL SIZE LAYOUT\nKEYS DIRECTLY TIED TO 74HC561\nPARALLEL-IN, SERIAL-OUT (PISO)\nSHIFT REGISTER FOR SCANNING"
+		(exclude_from_sim no)
+		(at 292.1 165.1 0)
 		(effects
 			(font
 				(size 2.54 2.54)
-			)
-		)
-	)
-	(text "12VDC\n500mA"
-		(exclude_from_sim no)
-		(at 165.1 76.2 0)
-		(effects
-			(font
-				(face "Comic Sans MS")
-				(size 1.27 1.27)
-			)
-		)
-	)
-	(text "3.3VDC\n500mA"
-		(exclude_from_sim no)
-		(at 234.442 76.2 0)
-		(effects
-			(font
-				(face "Comic Sans MS")
-				(size 1.27 1.27)
 			)
 		)
@@
 		)
 	)
-	(text "1.2VDC\n500mA"
-		(exclude_from_sim no)
-		(at 266.7 76.2 0)
-		(effects
-			(font
-				(face "Comic Sans MS")
-				(size 1.27 1.27)
+	(text "5VDC, 2A\n	TPS54231 BUCK CONVERTER\n	POWERS: APA102 LED's, USB2514 HUB\n3.3VDC, 1A\n	TPS62130 BUCK CONVERTER\n	POWERS: RM4A1 uC, STM32G431 uC, KEYS, E-INK"
+		(exclude_from_sim no)
+		(at 215.9 76.2 0)
+		(effects
+			(font
+				(size 2.54 2.54)
 			)
 		)
@@
 		)
 	)
-	(polyline
-		(pts
-			(xy 266.7 62.23) (xy 266.7 52.07)
-		)
-		(stroke
-			(width 0.381)
-			(type default)
-			(color 0 0 194 1)
-		)
-	)
-	(polyline
-		(pts
-			(xy 234.95 52.07) (xy 236.22 53.34)
+	(bus_entry
+		(at 63.5 -93.98)
+		(size 2.54 2.54)
+		(stroke
+			(width 0)
+			(type default)
+		)
+	)
+	(polyline
+		(pts
+			(xy 317.5 26.67) (xy 317.5 64.77)
+		)
+		(stroke
+			(width 0.381)
+			(type default)
+			(color 0 0 194 1)
+		)
+	)
+	(polyline
+		(pts
+			(xy 215.9 52.07) (xy 217.17 53.34)
 		)
 		(stroke
@@
 	(polyline
 		(pts
-			(xy 139.7 76.2) (xy 151.13 76.2)
-		)
-		(stroke
-			(width 0.381)
-			(type default)
-			(color 0 0 194 1)
-		)
-	)
-	(polyline
-		(pts
-			(xy 266.7 52.07) (xy 267.97 53.34)
-		)
-		(stroke
-			(width 0.381)
-			(type default)
-			(color 0 0 194 1)
-		)
-	)
-	(polyline
-		(pts
 			(xy 212.09 176.53) (xy 166.37 176.53)
 		)
@@
 	(polyline
 		(pts
-			(xy 265.43 53.34) (xy 266.7 52.07)
-		)
-		(stroke
-			(width 0.381)
-			(type default)
-			(color 0 0 194 1)
-		)
-	)
-	(polyline
-		(pts
-			(xy 133.35 54.61) (xy 196.85 54.61)
-		)
-		(stroke
-			(width 0.381)
-			(type default)
-			(color 0 0 194 1)
-		)
-	)
-	(polyline
-		(pts
 			(xy 220.98 138.43) (xy 220.98 176.53)
 		)
@@
 	(polyline
 		(pts
-			(xy 115.57 46.99) (xy 133.35 46.99)
-		)
-		(stroke
-			(width 0.381)
-			(type default)
-			(color 0 0 194 1)
-		)
-	)
-	(polyline
-		(pts
-			(xy 196.85 62.23) (xy 199.39 59.69)
+			(xy 327.66 63.5) (xy 328.93 64.77)
+		)
+		(stroke
+			(width 0.381)
+			(type default)
+			(color 0 0 194 1)
+		)
+	)
+	(polyline
+		(pts
+			(xy 115.57 46.99) (xy 127 46.99)
+		)
+		(stroke
+			(width 0.381)
+			(type default)
+			(color 0 0 194 1)
+		)
+	)
+	(polyline
+		(pts
+			(xy 149.86 76.2) (xy 147.32 73.66)
 		)
 		(stroke
@@
 	(polyline
 		(pts
-			(xy 254 63.5) (xy 254 88.9)
-		)
-		(stroke
-			(width 0)
-			(type default)
+			(xy 280.67 64.77) (xy 328.93 64.77)
+		)
+		(stroke
+			(width 0.381)
+			(type default)
+			(color 0 0 194 1)
 		)
 	)
@@
 	(polyline
 		(pts
-			(xy 215.9 63.5) (xy 215.9 88.9)
-		)
-		(stroke
-			(width 0)
-			(type default)
-		)
-	)
-	(polyline
-		(pts
 			(xy 148.59 35.56) (xy 151.13 38.1)
 		)
@@
 	(polyline
 		(pts
-			(xy 234.95 62.23) (xy 234.95 52.07)
+			(xy 215.9 62.23) (xy 215.9 52.07)
 		)
 		(stroke
@@
 	(polyline
 		(pts
+			(xy 328.93 64.77) (xy 327.66 66.04)
+		)
+		(stroke
+			(width 0.381)
+			(type default)
+			(color 0 0 194 1)
+		)
+	)
+	(polyline
+		(pts
 			(xy 353.06 111.76) (xy 355.6 114.3)
 		)
@@
 	(polyline
 		(pts
-			(xy 139.7 76.2) (xy 139.7 111.76)
+			(xy 127 54.61) (xy 127 113.03)
 		)
 		(stroke
@@
 	(polyline
 		(pts
+			(xy 327.66 25.4) (xy 328.93 26.67)
+		)
+		(stroke
+			(width 0.381)
+			(type default)
+			(color 0 0 194 1)
+		)
+	)
+	(polyline
+		(pts
 			(xy 166.37 203.2) (xy 168.91 205.74)
 		)
@@
 	(polyline
 		(pts
-			(xy 133.35 46.99) (xy 133.35 54.61)
+			(xy 127 46.99) (xy 127 54.61)
 		)
 		(stroke
@@
 	(polyline
 		(pts
-			(xy 194.31 59.69) (xy 196.85 62.23)
+			(xy 328.93 26.67) (xy 327.66 27.94)
+		)
+		(stroke
+			(width 0.381)
+			(type default)
+			(color 0 0 194 1)
+		)
+	)
+	(polyline
+		(pts
+			(xy 318.77 26.67) (xy 328.93 26.67)
+		)
+		(stroke
+			(width 0.381)
+			(type default)
+			(color 0 0 194 1)
+		)
+	)
+	(polyline
+		(pts
+			(xy 147.32 78.74) (xy 149.86 76.2)
 		)
 		(stroke
@@
 	(polyline
 		(pts
-			(xy 139.7 111.76) (xy 142.24 109.22)
-		)
-		(stroke
-			(width 0.381)
-			(type default)
-			(color 0 0 194 1)
-		)
-	)
-	(polyline
-		(pts
-			(xy 177.8 63.5) (xy 177.8 88.9)
-		)
-		(stroke
-			(width 0)
-			(type default)
+			(xy 127 113.03) (xy 129.54 110.49)
+		)
+		(stroke
+			(width 0.381)
+			(type default)
+			(color 0 0 194 1)
 		)
 	)
@@
 	(polyline
 		(pts
-			(xy 137.16 109.22) (xy 139.7 111.76)
+			(xy 124.46 110.49) (xy 127 113.03)
 		)
 		(stroke
@@
 	(polyline
 		(pts
-			(xy 233.68 53.34) (xy 234.95 52.07)
+			(xy 214.63 53.34) (xy 215.9 52.07)
+		)
+		(stroke
+			(width 0.381)
+			(type default)
+			(color 0 0 194 1)
+		)
+	)
+	(polyline
+		(pts
+			(xy 318.77 26.67) (xy 317.5 26.67)
 		)
 		(stroke
@@
 	(polyline
 		(pts
-			(xy 196.85 54.61) (xy 196.85 62.23)
-		)
-		(stroke
+			(xy 127 76.2) (xy 149.86 76.2)
+		)
+		(stroke
