File: Main/MicroController.kicad_sch (KiCad schematic)
At the start: 0 parts

Commit message: Add files via upload
Parts:
- added C32, C34, C39: 4.7uF, symbol Device:C_Small
- added C33, C35, C36, C38: 100nF, symbol Device:C_Small
- added C37: 1uF, symbol Device:C_Small
- added FB1, FB2: FerriteBead, symbol Device:FerriteBead
- added PB1: FSM2JELGELTR, symbol FSM2JELGELTR:FSM2JELGELTR
- added R30, R31: 5.1k, symbol Device:R_US
- added U8: R7FA4M1AB3CFM_AA0, R7FA4M1AB3CFM_AA0:QFP50P1200X1200X170-64N, symbol R7FA4M1AB3CFM_AA0:R7FA4M1AB3CFM_AA0
Connections:
- new net: PB1.3, PB1.4, R31.2, U8.25 (~{RES})
- new net: C39.1, U8.5 (VCL)
- new net: C38.1, FB2.1, U8.56 (AVCC0)
- new net: C37.1, FB1.2, U8.59 (P010/VREFH0)
- new net GND: C32.2, C33.2, C34.2, C35.2, C36.2, C37.2, C38.2, C39.2, PB1.1, PB1.2, PB1.5, U8.17 (VSS_USB), U8.40 (VSS__1), U8.57 (AVSS0), U8.8 (VSS)
- new net USB_OUT1_D+: U8.19 (P914/USB_DP)
- new net USB_OUT1_D-: U8.18 (P915/USB_DM)
- new net USB_VBUS1: C34.1, C35.1, C36.1, FB2.2, R30.1, R31.1, U8.11 (VCC), U8.21 (VCC_USB_LDO), U8.39 (VCC__1)
- new net uC_AREF: FB1.1, R30.2
- new net uC_VCC_USB: C32.1, C33.1, U8.20 (VCC_USB), U8.4 (VBATT)
