File: Main/Power Stage.kicad_sch (KiCad schematic)
At the start: 0 parts

Commit message: Add files via upload
Parts:
- added C10: .1uF, symbol Device:C_Small
- added C11, C12: 47uF, symbol Device:C_Small
- added C13: 1nF, symbol Device:C_Small
- added C14: 10pF, symbol Device:C_Small
- added C15, C8: 22uF, symbol Device:C_Small
- added C6: 10uF, symbol Device:C_Small
- added C7: 390pF, symbol Device:C_Small
- added C9: 8.2nF, symbol Device:C_Small
- added D4: SS24FL, symbol Device:D_Schottky
- added L1: SRN8040-8R2Y, symbol Device:L_Iron
- added L2: XGL5020-222MEC, symbol Device:L
- added R12: 10.2k, symbol Device:R_US
- added R13: 1.91k, symbol Device:R_US
- added R14: 169k, symbol Device:R_US
- added R15: 52.3k, symbol Device:R_US
- added R16: 28.7k, symbol Device:R_US
- added R17: 100k, symbol Device:R_US
- added R18: 562k, symbol Device:R_US
- added R19: 180k, symbol Device:R_US
- added U4: TPS54231DR, D8, symbol TPS54231DR:TPS54231DR
- added U5: TPS62130ARGTR, RGT0016C, symbol TPS62130ARGTR:TPS62130ARGTR
Connections:
- new net: R18.2, R19.1, U5.5 (FB)
- new net: R12.2, R13.1, U4.5 (VSENSE)
- new net: C10.1, D4.1 (K), L1.1, U4.8 (PH)
- new net: L2.1, U5.1 (SW), U5.2 (SW), U5.3 (SW)
- new net: R17.2, U5.4 (PG)
- new net: C7.1, U5.9 (SS_TR)
- new net: C10.2, U4.1 (BOOT)
- new net: C9.1, U4.4 (SS)
- new net: C14.1, R16.1, U4.6 (COMP)
- new net: C13.1, R16.2
- new net 3.3V_SYS: C15.1, L2.2, R17.1, R18.1, U5.14 (VOS), U5.7 (FSW)
- new net 5V_EN: R14.2, R15.1, U4.3 (EN)
- new net 5V_SYS: C11.1, C12.1, L1.2, R12.1
- new net GND: C11.2, C12.2, C13.2, C14.2, C15.2, C6.2, C7.2, C8.2, C9.2, D4.2 (A), R13.2, R15.2, R19.2, U4.7 (GND), U5.15 (PGND), U5.16 (PGND), U5.17 (EP), U5.6 (AGND), U5.8 (DEF)
- new net VBUS_SYS: C6.1, C8.1, R14.1, U4.2 (VIN), U5.10 (AVIN), U5.11 (PVIN), U5.12 (PVIN), U5.13 (EN)
