File: Main/Type C Output.kicad_sch (KiCad schematic)
At the start: 0 parts

Commit message: Add files via upload
Parts:
- added BR1: BGX50AE6327HTSA1, SOT143_2p9x1p3-1p9_INF, symbol BGX50AE6327HTSA1:BGX50AE6327HTSA1
- added C30: 1.0nF, symbol Device:C_Small
- added J2: 12402012E212A, 12402012E212A:AMPHENOL_12402012E212A, symbol 12402012E212A:12402012E212A
- added R28, R29: 5.1k, symbol Device:R_US
Connections:
- new net: J2.B5 (CC1_B), R28.1
- new net: J2.A5 (CC1_A), R29.1
- new net GND: BR1.3, C30.2, J2.A1_B12 (GND), J2.B1_A12 (GND__1), R28.2, R29.2
- new net GNDPWR: J2.SH1 (SHIELD), J2.SH2 (SHIELD__1), J2.SH3 (SHIELD__2), J2.SH4 (SHIELD__3)
- new net USB_OUT2_D+: BR1.2, J2.A6 (D+_A), J2.B6 (D+_B)
- new net USB_OUT2_D-: BR1.4, J2.A7 (D-_A), J2.B7 (D-_B)
- new net USB_VBUS2: BR1.1, C30.1, J2.A4_B9 (VBUS), J2.B4_A9 (VBUS__1)
- no-connect marks 0 -> 2
