File: Main/USB A Output.kicad_sch (KiCad schematic)
At the start: 0 parts

Commit message: Add files via upload
Parts:
- added BR2: BGX50AE6327HTSA1, SOT143_2p9x1p3-1p9_INF, symbol BGX50AE6327HTSA1:BGX50AE6327HTSA1
- added C31: 1.0nF, symbol Device:C_Small
- added J3: UE27AC54100, UE27AC54100:AMPHENOL_UE27AC54100, symbol UE27AC54100:UE27AC54100
Connections:
- new net GND: BR2.3, C31.2, J3.4 (GND)
- new net GNDPWR: J3.S1 (SHIELD), J3.S2 (SHIELD__1)
- new net USB_OUT3_D+: BR2.2, J3.3 (D+)
- new net USB_OUT3_D-: BR2.4, J3.2 (D-)
- new net USB_VBUS3: BR2.1, C31.1, J3.1 (VCC)
