File: Main/USB Hub.kicad_sch (KiCad schematic)
At the start: 3 parts, among them U3 USB2514B-AEZC

Commit message: Add files via upload
Parts:
- added C16, C17, C18, C19, C20, C21, C24, C25, C26, C27, C28: 0.1uF, symbol Device:C_Small
- added C22: 4.7uF, symbol Device:C_Small
- added C23: 1.0nF, symbol Device:C_Small
- added R20, R21, R22, R24: 100k, symbol Device:R_US
- added R23: 10k, symbol Device:R_US
- added R25: 12.0k 1%, symbol Device:R_US
- added R26: 1MEG, symbol Device:R_US
- added U6, U7: MIC2026-1YM, MIC2026-1YM:SOIC127P599X173-8N, symbol MIC2026-1YM:MIC2026-1YM
- added Y1: Crystal, symbol Device:Crystal
- R5, R6: value R_US -> 100k
Connections:
- net GND: now also C16.2, C17.2, C18.2, C19.2, C20.2, C21.2, C22.2, C23.2, C24.2, C25.2, C26.2, C27.1, C28.1, R20.2, R21.2, R22.2, R25.2, U6.6 (GND), U7.6 (GND)
- net 3.3V_SYS: now reaches U3.10 (VDDA33)
- net 3.3V_SYS: now also U3.15 (VDD33), U3.23 (VDD33), U3.29 (VDDA33), U3.36 (VDDA33), U3.5 (VDDA33), C16.1, C17.1, C18.1, C19.1, C20.1, C21.1, C22.1, R23.1, R24.1
- net USB_PRTPWR1: now reaches U3.12 (PRTPWR1/BC_EN1)
- net USB_PRTPWR1: now also U6.1 (ENA)
- net USB_OVRCRNT1: now reaches U3.13 (OCS_N1)
- net USB_OVRCRNT1: now also U6.2 (~{FLGA})
- net at U3.14 (CRFILT): now also C24.1
- net USB_PRTPWR2: now reaches U3.16 (PRTPWR2/BC_EN2)
- net USB_PRTPWR2: now also U6.4 (ENB)
- net USB_OVRCRNT2: now reaches U3.17 (OCS_N2)
- net USB_OVRCRNT2: now also U6.3 (~{FLGB})
- net USB_PRTPWR3: now reaches U3.18 (PRTPWR3/BC_EN3)
- net USB_PRTPWR3: now also U7.1 (ENA)
- net USB_OVRCRNT3: now reaches U3.19 (OCS_N3)
- net USB_OVRCRNT3: now also U7.2 (~{FLGA})
- net USB_PRTPWR4: now reaches U3.20 (PRTPWR4/BC_EN4)
- net USB_PRTPWR4: now also U7.4 (ENB)
- net USB_OVRCRNT4: now reaches U3.21 (OCS_N4)
- net USB_OVRCRNT4: now also U7.3 (~{FLGB})
- net at U3.22 (SDA/SMBDATA/NON_REM1): now also R20.1
- net at U3.24 (SCL/SMBCLK/CFG_SEL0): now also R21.1
- net at U3.25 (HS_IND/CFG_SEL1): now also R22.1
- net USB_RESET: now reaches U3.26 (RESET_N)
- net USB_RESET: now also C25.1, R24.2
- net at R5.2, R6.1, U3.27 (VBUS_DET): now also C23.1
- net at U3.28 (SUSP_IND/LOCAL_PWR/NON_REM0): now also R23.2
- net USB_XTAL2: now reaches U3.32 (XTALOUT)
- net USB_XTAL2: now also C28.2, R26.2, Y1.1
- net USB_XTAL1: now reaches U3.33 (XTALIN/CLKIN)
- net USB_XTAL1: now also C27.2, R26.1, Y1.2
- net at U3.34 (PLLFILT): now also C26.1
- net at U3.35 (RBIAS): now also R25.1
- net USB_OUT4_D-: now reaches U3.8 (USBDM_DN4/PRT_DIS_M4)
- net USB_OUT4_D+: now reaches U3.9 (USBDP_DN4/PRT_DIS_P4)
- net USB_DM renamed USB_IN_D-
- net USB_DP renamed USB_IN_D+
- net USB_OUT1_DM renamed USB_OUT1_D-
- net USB_OUT1_DP renamed USB_OUT1_D+
- net USB_OUT2_DM renamed USB_OUT2_D-
- net USB_OUT2_DP renamed USB_OUT2_D+
- net USB_OUT3_DM renamed USB_OUT3_D-
- net USB_OUT3_DP renamed USB_OUT3_D+
- net VBUS_SYS renamed 5V_SYS
- net 5V_SYS: now also U6.7 (IN), U7.7 (IN)
- new net USB_VBUS1: U6.8 (OUTA)
- new net USB_VBUS2: U6.5 (OUTB)
- new net USB_VBUS3: U7.8 (OUTA)
- new net USB_VBUS4: U7.5 (OUTB)
Other:
- note added: "NOTE 1: U3 IS STRAPPED TO CONFIGURE AS [0,0] FOR DEFAULT CONFIGURATION, NO INTERFACE CONNECTION. PORT 1 CONFIGURED AS NON-REMOVEABLE, WHICH WILL BE USED FOR RM4A1 uC CONNECTION."
- moved on the sheet: R5, R6, U3
